File: STM32G4.kicad_pcb (KiCad board)
At the start: 4 copper layers, 47.7 x 21.9 mm, 43 parts, among them J1 Conn_01x18, J2 Conn_01x18, J3 USB_C_Receptacle_USB2.0_16P, J4 Conn_01x04_Pin, SW1 RST_SW, SW2 RST_SW, U1 STM32G491CETx, U2 ICM-42688-P, U3 BMP280, U4 SPX3819M5-L-3-3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

Commit message: Second Commit
Parts:
- removed C10: 1uF, Capacitor_SMD:C_0402_1005Metric
- removed C9: .1uF, Capacitor_SMD:C_0402_1005Metric
- C1: footprint Capacitor_SMD:C_0402_1005Metric -> Capacitor_SMD:C_0201_0603Metric
- C12: footprint Capacitor_SMD:C_0603_1608Metric -> Capacitor_SMD:C_0402_1005Metric
- J1, J2: value Conn_01x18 -> Conn_01x15; footprint Connector_PinHeader_2.54mm:PinHeader_1x18_P2.54mm_Vertical -> Connector_PinHeader_2.54mm:PinHeader_1x15_P2.54mm_Vertical
- R7, R8: footprint Resistor_SMD:R_0402_1005Metric -> Resistor_SMD:R_0201_0603Metric
- moved C19 12.7 mm to (142.5, 76.0), turned to -90 degrees
- moved U3 10.6 mm to (144.4, 75.3), turned to 90 degrees
- moved R8 10.5 mm to (144.8, 73.3), turned to 180 degrees
- moved C20 10.5 mm to (146.7, 76.2), turned to 180 degrees
- moved R7 9.36 mm to (141.5, 75.2), turned to -90 degrees
- moved R6 5.73 mm to (121.5, 70.6), turned to 180 degrees
- moved R4 2.80 mm to (146.0, 65.0), turned to 180 degrees
- moved J1 2.54 mm to (154.9, 78.7)
- moved J2 2.54 mm to (154.9, 61.0)
- moved C1 1.92 mm to (137.6, 63.9), turned to -135 degrees
- moved FB1 1.79 mm to (131.2, 75.7), turned to 135 degrees
- moved C6 1.70 mm to (126.5, 64.6), turned to 90 degrees
- moved R2 1.66 mm to (151.6, 71.5), turned to 0 degrees
- moved C5 1.58 mm to (129.0, 67.8)
- moved R9 1.49 mm to (150.2, 76.0)
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Connections:
- J1 pad 10: /PB11 -> /PB12
- J1 pad 11: /PB10 -> /PB11
- J1 pad 12: /PB2 -> /PB10
- J1 pad 13: /PB1 -> /PB2
- J1 pad 14: /PB0 -> /PB1
- J1 pad 15: /MOSI -> GND
- J1 pad 3: /PA10 -> GND
- J1 pad 4: /PA9 -> /PA10
- J1 pad 5: /PA8 -> /I2C1_SCL
- J1 pad 6: /PB15 -> /I2C1_SDA
- J1 pad 7: /PB14 -> /PB15
- J1 pad 8: /PB13 -> /PB14
- J1 pad 9: /PB12 -> /PB13
- J2 pad 10: /PC14 -> NRST
- J2 pad 11: /PC15 -> /PA0
- J2 pad 12: NRST -> /PA1
- J2 pad 13: /PA0 -> /PA2
- J2 pad 14: /PA1 -> /PA3
- J2 pad 15: /PA2 -> GND
- J2 pad 2: /I2C1_SCL -> /PA15
- J2 pad 7: /I2C1_SDA -> /PB7
- U1 pad 12: /NSS -> /PA4
- U1 pad 16: /PB0 -> /NSS
- U1 pad 3: /PC14 -> unconnected-(U1-PC14-Pad3)
- U1 pad 30: /PA8 -> /I2C1_SDA
- U1 pad 31: /PA9 -> /I2C1_SCL
- U1 pad 39: /I2C1_SCL -> /PA15
- U1 pad 4: /PC15 -> unconnected-(U1-PC15-Pad4)
- U1 pad 44: /I2C1_SDA -> /PB7
- U2 pad 4: /PB0 -> /PA4
Routing:
- net +3.3V: track 18.7 -> 90.7 mm, vias 0 -> 14
- net GND: track 17.2 -> 50.5 mm, vias 10 -> 24
- net BOOT0: track 0.00 -> 33.3 mm, vias 0 -> 2
- net /SWDIO: track 0.00 -> 25.4 mm, vias 0 -> 1
- net NRST: track 0.00 -> 25.0 mm, vias 0 -> 3
- net /SWCLK: track 0.00 -> 24.4 mm, vias 0 -> 1
- net /PA3: track 0.00 -> 20.0 mm, vias 0 -> 2
- net /PC13: track 0.00 -> 16.3 mm, vias 0 -> 2
- net /PA2: track 0.00 -> 15.1 mm, vias 0 -> 2
- net VBUS: track 12.1 -> 27.0 mm, vias 3 -> 6
- net /PA15: track 0.00 -> 14.4 mm
- net /PB1: track 0.00 -> 14.1 mm
- net /PA10: track 0.00 -> 12.8 mm, vias 0 -> 1
- net /PB3: track 0.00 -> 12.1 mm
- net /PB2: track 0.00 -> 11.7 mm
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- added copper zone on F.Cu, net +3.3V
- added copper zone on F.Cu, net GND
Other:
- board size 47.7 x 21.9 mm -> 49.4 x 21.9 mm
